Commit message: initial edits for zalpiano URDF (incomplete)

File: odrive_demo_description/urdf/odrive.ros2_control.xacro (robot description, xacro)
@@ -1,6 +1,8 @@
 <?xml version="1.0"?>
 <robot xmlns:xacro="http://www.ros.org/wiki/xacro">
+  <!-- <xacro:macro name="odrive_ros2_control"
+    params="name serial_number:=^|000000000000 enable_joint0:=^|true enable_joint1:=^|true joint0_name:=^|joint0 joint1_name:=^|joint1"> -->
   <xacro:macro name="odrive_ros2_control"
-    params="name serial_number:=^|000000000000 enable_joint0:=^|true enable_joint1:=^|true joint0_name:=^|joint0 joint1_name:=^|joint1">
+    params="name serial_number:=^|357030673133 enable_joint0:=^|true enable_joint1:=^|true joint0_name:=^|drivewhl_l_joint joint1_name:=^|drivewhl_r_joint">
     <ros2_control name="${name}" type="system">
       <hardware>
@@ -15,5 +17,5 @@
           <param name="axis">0</param>
           <param name="enable_watchdog">1</param>
-          <param name="watchdog_timeout">0.1</param>
+          <param name="watchdog_timeout">0.5</param>
         </joint>
       </xacro:if>
@@ -23,5 +25,5 @@
           <param name="axis">1</param>
           <param name="enable_watchdog">1</param>
-          <param name="watchdog_timeout">0.1</param>
+          <param name="watchdog_timeout">0.5</param>
         </joint>
       </xacro:if>

File: odrive_demo_description/urdf/odrive_diffbot.urdf.xacro (robot description, xacro)
@@ -2,11 +2,17 @@
 <robot xmlns:xacro="http://www.ros.org/wiki/xacro" name="diffdrive_robot">
   <xacro:arg name="prefix" default="" />
-  <xacro:include filename="$(find diffbot_description)/urdf/diffbot_description.urdf.xacro" />
-  <xacro:include filename="$(find diffbot_description)/gazebo/diffbot.materials.xacro" />
+  <!-- <xacro:include filename="$(find diffbot_description)/urdf/diffbot_description.urdf.xacro" /> -->
+  <xacro:include filename="$(find zalpiano_desc)/src/description/zalpiano_description.urdf.xacro" />
+  <!-- <xacro:include filename="$(find diffbot_description)/gazebo/diffbot.materials.xacro" /> -->
+  <!-- We don't need to have materials defined for the zalpiano_desc.urdf.xacro -->
   <xacro:include filename="$(find odrive_demo_description)/urdf/odrive.ros2_control.xacro" />
   <xacro:diffbot prefix="$(arg prefix)" />
+  <!-- <xacro:odrive_ros2_control
+    name="ODriveDiffBot"
+    joint0_name="$(arg prefix)left_wheel_joint"
+    joint1_name="$(arg prefix)right_wheel_joint" /> -->
   <xacro:odrive_ros2_control
     name="ODriveDiffBot"
-    joint0_name="$(arg prefix)left_wheel_joint"
-    joint1_name="$(arg prefix)right_wheel_joint" />
+    joint0_name="$(arg prefix)drivewhl_l_joint"
+    joint1_name="$(arg prefix)drivewhl_r_joint" />
 </robot>
