Commit message: added aruco marker joints (links). TODO: measure accurate wheel separationdistance to put into diffbot_controllers.yaml

File: zalpiano_desc/src/description/zalpiano_description.urdf.xacro (robot description, xacro)
@@ -94,3 +94,103 @@
     <origin xyz="${-caster_xoff} 0.0 ${-(base_height/2)}" rpy="0 0 0"/>
   </joint>
+  <!-- ////////////////////////////////////////////////////// -->
+  <!-- ////////////////////////////////////////////////////// -->
+  <!-- ////////////////////////////////////////////////////// -->
+  <!-- ////////////////////////////////////////////////////// -->
+  <!-- ArUco Marker 0 -->
+  <link name="aruco_marker_0_link">
+    <visual>
+      <origin xyz="0 0 0.001" rpy="0 0 -1.5709"/>
+      <geometry>
+        <box size="0.09 0.09 0.001"/>
+      </geometry>
+      <material name="Aruco0">
+        <!-- color for RVIZ-->
+        <color rgba="1 1 0 1"/>
+      </material>
+    </visual>
+    <collision>
+      <origin xyz="0 0 0.001" rpy="0 0 -1.5709"/>
+      <geometry>
+        <box size="0.09 0.09 0.001"/>
+      </geometry>
+    </collision>
+  </link>
+  <joint name="base_to_aruco_marker_0" type="fixed">
+    <parent link="base_link"/>
+    <child link="aruco_marker_0_link"/>
+    <origin xyz="0.1 0 ${(base_height)/2}" rpy="0 0 -1.5709"/>
+  </joint>
+  <!-- ArUco Marker 1 -->
+  <link name="aruco_marker_1_link">
+    <visual>
+      <origin xyz="0 0 0.001" rpy="0 0 -1.5709"/>
+      <geometry>
+        <box size="0.09 0.09 0.001"/>
+      </geometry>
+      <material name="Aruco1">
+        <!-- color for RVIZ-->
+        <color rgba="1 0 0 1"/>
+      </material>
+    </visual>
+    <collision>
+      <origin xyz="0 0 0.001" rpy="0 0 -1.5709"/>
+      <geometry>
+        <box size="0.09 0.09 0.001"/>
+      </geometry>
+    </collision>
+  </link>
+  <joint name="base_to_aruco_marker_1" type="fixed">
+    <parent link="base_link"/>
+    <child link="aruco_marker_1_link"/>
+    <origin xyz="0 0.1 ${(base_height)/2}" rpy="0 0 -1.5709"/>
+  </joint>
+  <!-- ArUco Marker 2 -->
+  <link name="aruco_marker_2_link">
+    <visual>
+      <origin xyz="0 0 0.001" rpy="0 0 -1.5709"/>
+      <geometry>
+        <box size="0.09 0.09 0.001"/>
+      </geometry>
+      <material name="Aruco2">
+        <!-- color for RVIZ-->
+        <color rgba="1 0 0 1"/>
+      </material>
+    </visual>
+    <collision>
+      <origin xyz="0 0 0.001" rpy="0 0 -1.5709"/>
+      <geometry>
+        <box size="0.09 0.09 0.001"/>
+      </geometry>
+    </collision>
+  </link>
+  <joint name="base_to_aruco_marker_2" type="fixed">
+    <parent link="base_link"/>
+    <child link="aruco_marker_2_link"/>
+    <origin xyz="-0.1 0 ${(base_height)/2}" rpy="0 0 -1.5709"/>
+  </joint>
+  <!-- ArUco Marker 3 -->
+  <link name="aruco_marker_3_link">
+    <visual>
+      <origin xyz="0 0 0.001" rpy="0 0 -1.5709"/>
+      <geometry>
+        <box size="0.09 0.09 0.001"/>
+      </geometry>
+      <material name="Aruco3">
+        <!-- color for RVIZ-->
+        <color rgba="1 0 0 1"/>
+      </material>
+    </visual>
+    <collision>
+      <origin xyz="0 0 0.001" rpy="0 0 -1.5709"/>
+      <geometry>
+        <box size="0.09 0.09 0.001"/>
+      </geometry>
+    </collision>
+  </link>
+  <joint name="base_to_aruco_marker_3" type="fixed">
+    <parent link="base_link"/>
+    <child link="aruco_marker_3_link"/>
+    <origin xyz="0 -0.1 ${(base_height)/2}" rpy="0 0 -1.5709"/>
+  </joint>
 </robot>

Commit message: added aruco center transforms and image topic publisher from real camera

File: zalpiano_desc/src/description/zalpiano_description.urdf.xacro (robot description, xacro)
@@ -194,3 +194,35 @@
     <origin xyz="0 -0.1 ${(base_height)/2}" rpy="0 0 -1.5709"/>
   </joint>
+  <!-- ////////////////////////////////////////////////////// -->
+  <!-- ////////////////////////////////////////////////////// -->
+  <!-- ////////////////////////////////////////////////////// -->
+  <!-- ////////////////////////////////////////////////////// -->
+  <link name="aruco_center_link0">
+  </link>
+  <joint name="center_to_aruco_marker_0" type="fixed">
+    <parent link="base_link"/>
+    <child link="aruco_center_link0"/>
+    <origin xyz="0 0 0" rpy="0 0 0"/>
+  </joint>
+  <link name="aruco_center_link1">
+  </link>
+  <joint name="center_to_aruco_marker_1" type="fixed">
+    <parent link="base_link"/>
+    <child link="aruco_center_link1"/>
+    <origin xyz="0 0 0" rpy="0 0 0"/>
+  </joint>
+  <link name="aruco_center_link2">
+  </link>
+  <joint name="center_to_aruco_marker_2" type="fixed">
+    <parent link="base_link"/>
+    <child link="aruco_center_link2"/>
+    <origin xyz="0 0 0" rpy="0 0 0"/>
+  </joint>
+  <link name="aruco_center_link3">
+  </link>
+  <joint name="center_to_aruco_marker_3" type="fixed">
+    <parent link="base_link"/>
+    <child link="aruco_center_link3"/>
+    <origin xyz="0 0 0" rpy="0 0 0"/>
+  </joint>
 </robot>

Commit message: fix some errors with aruco rotation, etc.

File: zalpiano_desc/src/description/zalpiano_description.urdf.xacro (robot description, xacro)
@@ -103,5 +103,5 @@
       <origin xyz="0 0 0.001" rpy="0 0 -1.5709"/>
       <geometry>
-        <box size="0.09 0.09 0.001"/>
+        <box size="0.1 0.1 0.001"/>
       </geometry>
       <material name="Aruco0">
@@ -113,5 +113,5 @@
       <origin xyz="0 0 0.001" rpy="0 0 -1.5709"/>
       <geometry>
-        <box size="0.09 0.09 0.001"/>
+        <box size="0.1 0.1 0.001"/>
       </geometry>
     </collision>
@@ -120,5 +120,5 @@
     <parent link="base_link"/>
     <child link="aruco_marker_0_link"/>
-    <origin xyz="0.1 0 ${(base_height)/2}" rpy="0 0 -1.5709"/>
+    <origin xyz="0.15 0 ${(base_height)/2}" rpy="0 0 -1.5709"/>
   </joint>
   <!-- ArUco Marker 1 -->
@@ -127,5 +127,5 @@
       <origin xyz="0 0 0.001" rpy="0 0 -1.5709"/>
       <geometry>
-        <box size="0.09 0.09 0.001"/>
+        <box size="0.1 0.1 0.001"/>
       </geometry>
       <material name="Aruco1">
@@ -137,5 +137,5 @@
       <origin xyz="0 0 0.001" rpy="0 0 -1.5709"/>
       <geometry>
-        <box size="0.09 0.09 0.001"/>
+        <box size="0.1 0.1 0.001"/>
       </geometry>
     </collision>
@@ -144,5 +144,5 @@
     <parent link="base_link"/>
     <child link="aruco_marker_1_link"/>
-    <origin xyz="0 0.1 ${(base_height)/2}" rpy="0 0 -1.5709"/>
+    <origin xyz="0 0.15 ${(base_height)/2}" rpy="0 0 -1.5709"/>
   </joint>
   <!-- ArUco Marker 2 -->
@@ -151,5 +151,5 @@
       <origin xyz="0 0 0.001" rpy="0 0 -1.5709"/>
       <geometry>
-        <box size="0.09 0.09 0.001"/>
+        <box size="0.1 0.1 0.001"/>
       </geometry>
       <material name="Aruco2">
@@ -161,5 +161,5 @@
       <origin xyz="0 0 0.001" rpy="0 0 -1.5709"/>
       <geometry>
-        <box size="0.09 0.09 0.001"/>
+        <box size="0.1 0.1 0.001"/>
       </geometry>
     </collision>
@@ -168,5 +168,5 @@
     <parent link="base_link"/>
     <child link="aruco_marker_2_link"/>
-    <origin xyz="-0.1 0 ${(base_height)/2}" rpy="0 0 -1.5709"/>
+    <origin xyz="-0.15 0 ${(base_height)/2}" rpy="0 0 -1.5709"/>
   </joint>
   <!-- ArUco Marker 3 -->
@@ -175,5 +175,5 @@
       <origin xyz="0 0 0.001" rpy="0 0 -1.5709"/>
       <geometry>
-        <box size="0.09 0.09 0.001"/>
+        <box size="0.1 0.1 0.001"/>
       </geometry>
       <material name="Aruco3">
@@ -185,5 +185,5 @@
       <origin xyz="0 0 0.001" rpy="0 0 -1.5709"/>
       <geometry>
-        <box size="0.09 0.09 0.001"/>
+        <box size="0.1 0.1 0.001"/>
       </geometry>
     </collision>
@@ -192,5 +192,5 @@
     <parent link="base_link"/>
     <child link="aruco_marker_3_link"/>
-    <origin xyz="0 -0.1 ${(base_height)/2}" rpy="0 0 -1.5709"/>
+    <origin xyz="0 -0.15 ${(base_height)/2}" rpy="0 0 -1.5709"/>
   </joint>
   <!-- ////////////////////////////////////////////////////// -->
@@ -203,5 +203,5 @@
     <parent link="base_link"/>
     <child link="aruco_center_link0"/>
-    <origin xyz="0 0 0" rpy="0 0 0"/>
+    <origin xyz="0 0 0" rpy="0 0 -1.5709"/>
   </joint>
   <link name="aruco_center_link1">
@@ -210,5 +210,5 @@
     <parent link="base_link"/>
     <child link="aruco_center_link1"/>
-    <origin xyz="0 0 0" rpy="0 0 0"/>
+    <origin xyz="0 0 0" rpy="0 0 -1.5709"/>
   </joint>
   <link name="aruco_center_link2">
@@ -217,5 +217,5 @@
     <parent link="base_link"/>
     <child link="aruco_center_link2"/>
-    <origin xyz="0 0 0" rpy="0 0 0"/>
+    <origin xyz="0 0 0" rpy="0 0 -1.5709"/>
   </joint>
   <link name="aruco_center_link3">
@@ -224,5 +224,5 @@
     <parent link="base_link"/>
     <child link="aruco_center_link3"/>
-    <origin xyz="0 0 0" rpy="0 0 0"/>
+    <origin xyz="0 0 0" rpy="0 0 -1.5709"/>
   </joint>
 </robot>

Commit message: debug aruco marker pose

File: zalpiano_desc/src/description/zalpiano_description.urdf.xacro (robot description, xacro)
@@ -101,5 +101,5 @@
   <link name="aruco_marker_0_link">
     <visual>
-      <origin xyz="0 0 0.001" rpy="0 0 -1.5709"/>
+      <origin xyz="0 0 0.001" rpy="0 0 0"/>
       <geometry>
         <box size="0.1 0.1 0.001"/>
@@ -111,5 +111,5 @@
     </visual>
     <collision>
-      <origin xyz="0 0 0.001" rpy="0 0 -1.5709"/>
+      <origin xyz="0 0 0.001" rpy="0 0 0"/>
       <geometry>
         <box size="0.1 0.1 0.001"/>
@@ -120,10 +120,10 @@
     <parent link="base_link"/>
     <child link="aruco_marker_0_link"/>
-    <origin xyz="0.15 0 ${(base_height)/2}" rpy="0 0 -1.5709"/>
+    <origin xyz="0.185 0 ${(base_height)/2}" rpy="0 0 0"/>
   </joint>
   <!-- ArUco Marker 1 -->
   <link name="aruco_marker_1_link">
     <visual>
-      <origin xyz="0 0 0.001" rpy="0 0 -1.5709"/>
+      <origin xyz="0 0 0.001" rpy="0 0 0"/>
       <geometry>
         <box size="0.1 0.1 0.001"/>
@@ -135,5 +135,5 @@
     </visual>
     <collision>
-      <origin xyz="0 0 0.001" rpy="0 0 -1.5709"/>
+      <origin xyz="0 0 0.001" rpy="0 0 0"/>
       <geometry>
         <box size="0.1 0.1 0.001"/>
@@ -144,10 +144,10 @@
     <parent link="base_link"/>
     <child link="aruco_marker_1_link"/>
-    <origin xyz="0 0.15 ${(base_height)/2}" rpy="0 0 -1.5709"/>
+    <origin xyz="0 0.185 ${(base_height)/2}" rpy="0 0 0"/>
   </joint>
   <!-- ArUco Marker 2 -->
   <link name="aruco_marker_2_link">
     <visual>
-      <origin xyz="0 0 0.001" rpy="0 0 -1.5709"/>
+      <origin xyz="0 0 0.001" rpy="0 0 0"/>
       <geometry>
         <box size="0.1 0.1 0.001"/>
@@ -159,5 +159,5 @@
     </visual>
     <collision>
-      <origin xyz="0 0 0.001" rpy="0 0 -1.5709"/>
+      <origin xyz="0 0 0.001" rpy="0 0 0"/>
       <geometry>
         <box size="0.1 0.1 0.001"/>
@@ -168,10 +168,10 @@
     <parent link="base_link"/>
     <child link="aruco_marker_2_link"/>
-    <origin xyz="-0.15 0 ${(base_height)/2}" rpy="0 0 -1.5709"/>
+    <origin xyz="-0.185 0 ${(base_height)/2}" rpy="0 0 0"/>
   </joint>
   <!-- ArUco Marker 3 -->
   <link name="aruco_marker_3_link">
     <visual>
-      <origin xyz="0 0 0.001" rpy="0 0 -1.5709"/>
+      <origin xyz="0 0 0.001" rpy="0 0 0"/>
       <geometry>
         <box size="0.1 0.1 0.001"/>
@@ -183,5 +183,5 @@
     </visual>
     <collision>
-      <origin xyz="0 0 0.001" rpy="0 0 -1.5709"/>
+      <origin xyz="0 0 0.001" rpy="0 0 0"/>
       <geometry>
         <box size="0.1 0.1 0.001"/>
@@ -192,5 +192,5 @@
     <parent link="base_link"/>
     <child link="aruco_marker_3_link"/>
-    <origin xyz="0 -0.15 ${(base_height)/2}" rpy="0 0 -1.5709"/>
+    <origin xyz="0 -0.185 ${(base_height)/2}" rpy="0 0 0"/>
   </joint>
   <!-- ////////////////////////////////////////////////////// -->
@@ -203,5 +203,5 @@
     <parent link="base_link"/>
     <child link="aruco_center_link0"/>
-    <origin xyz="0 0 0" rpy="0 0 -1.5709"/>
+    <origin xyz="0 0 0" rpy="0 0 0"/>
   </joint>
   <link name="aruco_center_link1">
@@ -210,5 +210,5 @@
     <parent link="base_link"/>
     <child link="aruco_center_link1"/>
-    <origin xyz="0 0 0" rpy="0 0 -1.5709"/>
+    <origin xyz="0 0 0" rpy="0 0 0"/>
   </joint>
   <link name="aruco_center_link2">
@@ -217,5 +217,5 @@
     <parent link="base_link"/>
     <child link="aruco_center_link2"/>
-    <origin xyz="0 0 0" rpy="0 0 -1.5709"/>
+    <origin xyz="0 0 0" rpy="0 0 0"/>
   </joint>
   <link name="aruco_center_link3">
@@ -224,5 +224,5 @@
     <parent link="base_link"/>
     <child link="aruco_center_link3"/>
-    <origin xyz="0 0 0" rpy="0 0 -1.5709"/>
+    <origin xyz="0 0 0" rpy="0 0 0"/>
   </joint>
 </robot>
